File: pcb/smd/zeta2/zeta2.sch (EAGLE design)
At the start: 126 parts, among them IC1 MAX6520, IC2 L293DD, IC3 L293DD, IC4 ULN2003AD, Q9 8MHz, U1 MPU-6050, U2 INA219, U3 ADS1115, U4 INA219, U5 DS18B20U+

Commit message: added i2c device
Parts:
- removed 3V3_OUT, 5V_OUT, 8V_OUT, FAN: JST-PH_2-PIN_HEADER, srg:JST-PH_2-PIN_HEADER
- removed ANALOG1, ANALOG2, EX_IO, HALL_SENSOR_A1120, LED, ONE_WIRE: JST-PH_3-PIN_HEADER, srg:JST-PH_3-PIN_HEADER
- removed C10, C13: 0.1µF, rcl:CPOL-EUSMCA
- removed C12, C34, C43: 47µF, rcl:CPOL-EUSMCC
- removed C14: 100µF, rcl:CPOL-EUSMCC
- removed C15: 100nF, rcl:C-EUC0603
- removed C17: 2,2nF, rcl:C-EUC0603
- removed C18, C19, C20, C21, C3, C32, C35, C42, C44: 0.1µF, rcl:C-EUC0603
- removed C2, C22: 4.7µF, rcl:C-EUC0603
- removed C30, C31, C33, C38, C39, C40, C41: 10nF, rcl:C-EUC0603
- removed C36, C37: 10µF, rcl:C-EUC0603
- removed D3: 1N4004 SMD, diode:DIODE-MELF-MLL41
- removed I2C, MOTOR_LEFT, RGB_LED, TFMINI: JST-PH_4-PIN_HEADER, srg:JST-PH_4-PIN_HEADER
- removed IC3: L293DD, st-microelectronics:L293DD
- removed IC4: ULN2003AD, uln-udn:ULN2003AD
- removed IRLML2502: (no value), zetex:NMOSSOT23
- removed JP3, JP4: (no value), jumper:JP2E
- removed J_MOTOR_DRIVER_1: MOTOR_DRIVER, Pololu Encoder and Motor Driver:MOTOR_DRIVER
- removed MICRO_USB_B: 47346-0001, 47346-0001:47346-0001
- removed PCA9306: (no value), srg:IC2_LEVEL_TRANSLATER
- removed PI_HEADER: (no value), con-lsta:FE20-2
- removed Q5: (no value), semicon-smd-ipc:PNP-TRANSISTOR_SOT23
- removed Q6, Q8: (no value), semicon-smd-ipc:NPN-TRANSISTOR_SOT23
- removed Q9: 8MHz, crystal-geyer_V1_0:KX-13
- removed R12, R14, R22, R31, R32, R33, R8: 100k, rcl:R-EU_R0603
- removed R13, R5, R6: 500R, rcl:R-EU_R0603
- removed R15, R16, R23, R24: 5k, rcl:R-EU_R0603
- removed R19, R20, R21: 22R, rcl:R-EU_R0603
- removed R25, R26, R27, R28, R29: 220R, rcl:R-EU_R0603
- removed R30: 4k7, rcl:R-EU_R0603
- removed SJ2: (no value), jumper:SJ2W
- removed SJ3, SJ4, SJ5: (no value), microbuilder:SOLDERJUMPERREFLOW_NOPASTE
- removed U$2: HMC5883L, HMC5883L:HMC5883L
- removed U$3: BMP085, BMP085:BMP085
- removed U1: MPU-6050, MPU-6050:MPU-6050
- removed U3: ADS1115, ADS1115:ADS1115
- removed U5: DS18B20U+, DS18B20U_:DS18B20U+
- C1: value 0.22µF -> 0.1nF
- U$1: value STM32F103C8T6 -> RPI-ZERO; device STM32F103C8T6:STM32F103C8T6 -> rpi-zero:RPI-ZERO
Connections:
- removed net ANALOG_3V3: HALL_SENSOR_A1120.2, U$1.PA0
- removed net A_RDY: U3.ALERT/RDY
- removed net BMP_EOC: U$3.EOC
- removed net BOOT0: JP3.2, PI_HEADER.29, R31.2, U$1.BOOT0
- removed net BOOT1: JP4.2, PI_HEADER.27, R33.1, U$1.PB2
- removed net HMC_RDY: U$2.DRDY
- removed net LED_1: IC4.I4
- removed net LED_2: IC4.I3
- removed net LED_B: IC4.I5
- removed net LED_G: IC4.I6
- removed net LED_R: IC4.I7
- removed net MPU_INT: U1.INT
- removed net M_DIR_2: R13.1, R5.1
- removed net N$13: Q5.B, R5.2
- removed net N$14: Q6.B, R6.2
- removed net N$15: Q8.B, R13.2
- removed net N$16: C17.1, U1.CPOUT
- removed net N$19: C21.1, U1.REGOUT
- removed net N$2: C1.2, U$2.SETC
- removed net N$23: C31.1, IC3.OUT3, MOTOR_LEFT.3
- removed net N$24: C31.2, IC3.OUT4, MOTOR_LEFT.4
- removed net N$25: C30.2, IC3.OUT2, MOTOR_LEFT.2
- removed net N$26: C30.1, IC3.OUT1, MOTOR_LEFT.1
- removed net N$27: IC4.O7, R29.1
- removed net N$28: C36.2, Q9.1, U$1.OSC_OUT
- removed net N$29: C37.2, Q9.2, U$1.OSC_IN
- removed net N$3: C1.1, U$2.SETP
- removed net N$30: IRLML2502.G, R21.2
- removed net N$31: IC4.O6, R25.1
- removed net N$32: R20.1, U$1.PA11
- removed net N$33: R19.1, U$1.PA12
- removed net N$34: R22.1, U$1.PC13-TAMPER-RTC
- removed net N$35: PI_HEADER.37, SJ3.2
- removed net N$36: PI_HEADER.35, SJ4.2
- removed net N$37: IC4.O5, R26.1
- removed net N$38: I2C.1, PCA9306.ENABLE, PCA9306.VREF2, R23.2, R24.2, SJ2.2
- removed net N$39: I2C.2, PCA9306.SCL2, R23.1
- removed net N$4: C2.1, U$2.C1
- removed net N$40: I2C.3, PCA9306.SDA2, R24.1
- removed net N$41: IC4.O4, R27.1
- removed net N$42: IC4.O3, R28.1
- removed net N$43: MICRO_USB_B.ID, R32.2
- removed net N$44: LED.1, R28.2
- removed net N$45: R29.2, RGB_LED.3
- removed net N$46: R25.2, RGB_LED.2
- removed net N$47: R26.2, RGB_LED.1
- removed net N$48: LED.2, R27.2
- removed net N$49: MICRO_USB_B.VBUS, SJ5.2
- removed net N$50: ANALOG1.2, U3.AIN0
- removed net N$51: ANALOG2.2, U3.AIN2
- removed net N$55: C41.2, D3.A, FAN.2, IRLML2502.D
- removed net N$6: IC3.IN2, IC3.IN3, Q8.C, R8.1
- removed net N$7: IC3.IN1, IC3.IN4, Q5.C, R14.2
- removed net N$9: IC3.EN1, IC3.EN2, Q6.C, R12.1
- removed net NRST: PI_HEADER.26, U$1.NRST
- removed net PIN_OUT: EX_IO.2, U$1.PB15
- removed net PWM_FAN: R21.1
- removed net PWM_M_EN_2: R6.1, U$1.PB0
- removed net SWCLK: PI_HEADER.20
- removed net SWDCLK: U$1.PA14
- removed net SWDIO: PI_HEADER.24, U$1.PA13
- removed net S_DIR: U$1.PA4
- removed net S_PWM_SPEED: U$1.PB1
- removed net TEMPERATURE: ONE_WIRE.2, R30.1, U5.DQ
- removed net USART1_RX: TFMINI.3, U$1.PA10
- removed net USART1_TX: TFMINI.2, U$1.PA9
- removed net USART2_RX: PI_HEADER.34, U$1.PA3
- removed net USART2_TX: PI_HEADER.32, U$1.PA2
- removed net USB_DM: MICRO_USB_B.D-, R20.2
- removed net USB_DP: MICRO_USB_B.D+, R19.2
- net +3V3: no longer 3V3_OUT.1, C15.1, C18.1, C20.1, C22.1, C32.1, C33.1, C38.1, C39.1, C40.1, C44.1, HALL_SENSOR_A1120.1, JP3.1, JP4.1, ONE_WIRE.1, PCA9306.VREF1, R15.1, R16.1, R30.2, R31.1, SJ2.1, U$1.VDD1, U$1.VDD2, U$1.VDD3, U$1.VDDA, U$2.S1, U$2.VDD, U$2.VDDIO, U$3.VDDA, U$3.VDDD, U1.VDD, U1.VLOGIC, U3.VDD, U5.VDD
- net +5V: now also C1.1; no longer 5V_OUT.1, ANALOG1.1, ANALOG2.1, C10.+, C13.+, C14.+, C19.1, C3.1, C34.+, C42.1, EX_IO.1, IC3.VSS, IC4.CD+, PI_HEADER.38, PI_HEADER.40, Q5.E, R12.2, R8.2, SJ2.3, SJ5.1, TFMINI.1
- net +8V: no longer 8V_OUT.1, C12.+, C35.1, C41.1, C43.+, D3.C, FAN.1, IC3.VS
- net GND: now also C1.2, U$10.IN-; no longer 3V3_OUT.2, 5V_OUT.2, 8V_OUT.2, ANALOG1.3, ANALOG2.3, C10.-, C12.-, C13.-, C14.-, C15.2, C17.2, C18.2, C19.2, C2.2, C20.2, C21.2, C22.2, C3.2, C32.2, C33.2, C34.-, C35.2, C36.1, C37.1, C38.2, C39.2, C40.2, C42.2, C43.-, C44.2, EX_IO.3, HALL_SENSOR_A1120.3, I2C.4, IC3.GND@1, IC3.GND@2, IC3.GND@3, IC3.GND@4, IC3.GND@5, IC3.GND@6, IC3.GND@7, IC3.GND@8, IC4.GND, IRLML2502.S, JP3.3, JP4.3, LED.3, MICRO_USB_B.GND, MICRO_USB_B.SHIELD, ONE_WIRE.3, PCA9306.GND, PI_HEADER.1, PI_HEADER.12, PI_HEADER.15, PI_HEADER.22, PI_HEADER.28, PI_HEADER.31, PI_HEADER.36, PI_HEADER.8, Q6.E, Q8.E, R14.1, R22.2, R32.1, R33.2, RGB_LED.4, TFMINI.4, U$1.VSS1, U$1.VSS2, U$1.VSS3, U$1.VSSA, U$10.IN+, U$2.GND, U$3.GND, U$3.XCLR, U1.AD0, U1.CLKIN, U1.FSYNC, U1.GND, U3.ADDR, U3.AIN1, U3.AIN3, U3.VSS, U5.GND
- net M_DIR_1: no longer U$1.PA5, U$1.PA7
- net N$17: now also MOTOR_RIGHT.4; no longer MOTOR_RIGHT.3
- net N$18: now also MOTOR_RIGHT.3; no longer MOTOR_RIGHT.4
- net N$20: now also MOTOR_RIGHT.1; no longer MOTOR_RIGHT.2
- net N$21: now also MOTOR_RIGHT.2; no longer MOTOR_RIGHT.1
- net PWM_M_EN_1: no longer U$1.PA6
- net SCL: no longer PCA9306.SCL1, R15.2, SJ4.1, U$1.PB6, U$2.SCL, U$3.SCL, U1.SCL, U3.SCL
- net SDA: no longer PCA9306.SDA1, R16.2, SJ3.1, U$1.PB7, U$2.SDA, U$3.SDA, U1.SDA, U3.SDA
- net V+: now also U$10.IN+; no longer U$10.IN-
Other:
- moved on the sheet: C1, C11, C23, C24, C25, C26, C28, C29, C4, C5, C6, C7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
