File: pcb/smd/zeta2/zeta2rework_lw_v5.sch (EAGLE design)
At the start: 104 parts, among them IC1 MAX6520, IC2 L293DD, IC3 L293DD, Q12 8MHz, U1 MPU-6050, U2 INA219, U5 DS18B20U+

Commit message: finished pcb
Parts:
- added U$2: RPI-ZERO, rpi-zero:RPI-ZERO
Changed lines of the file:
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@@
 <part name="+3V1" library="supply1" library_urn="urn:adsk.eagle:library:371" deviceset="+3V3" device=""/>
 <part name="C11" library="rcl" library_urn="urn:adsk.eagle:library:334" deviceset="C-EU" device="C1206" package3d_urn="urn:adsk.eagle:package:23618/2" value="0.1µF"/>
+<part name="U$2" library="rpi-zero" deviceset="RPI-ZERO" device=""/>
 </parts>
 <sheets>
@@
 <instance part="+3V1" gate="G$1" x="86.36" y="-10.16"/>
 <instance part="C11" gate="G$1" x="292.1" y="-40.64"/>
+<instance part="U$2" gate="G$1" x="-182.88" y="-66.04"/>
 </instances>
 <busses>
