File: pcb/smd/zeta2/zeta2rework_lw_v6.brd (EAGLE design)
At the start: 80.3 x 43.2 mm, 104 parts, among them IC1 MAX6520, IC2 L293DD, IC3 L293DD, Q12 8MHz, U1 MPU-6050, U2 INA219, U5 DS18B20U+

Commit message: finished pcb
Parts:
- added IC4: TLC59711, adafruit:HTSSOP20DAP
- flipped U$10 to the bottom, turned to 180 degrees
Connections:
- new net VCC: IC4.19
- net GND: now also IC4.2
Routing:
- net GND: track 226.0 -> 233.9 mm, vias 2 -> 3
- net +8V: track 58.3 -> 56.3 mm
Changed lines of the file:
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@@
 <drawing>
 <settings>
-<setting alwaysvectorfont="yes"/>
+<setting alwaysvectorfont="no"/>
 <setting verticaltext="up"/>
 </settings>
@@
 <attribute name="SPICEPREFIX" value="C" x="4.445" y="12.065" size="1.778" layer="27" rot="R270" display="off"/>
 </element>
-<element name="U$10" library="diy-modules" package="DC-DC-STEP-DOWN-MP2307" value="DC-DC-STEP-DOWN-MP2307" x="23.495" y="15.24"/>
+<element name="U$10" library="diy-modules" package="DC-DC-STEP-DOWN-MP2307" value="DC-DC-STEP-DOWN-MP2307" x="23.495" y="15.24" rot="MR180"/>
 <element name="C16" library="rcl" library_urn="urn:adsk.eagle:library:334" package="C1206" package3d_urn="urn:adsk.eagle:package:23618/2" value="0.1µF" x="8.255" y="12.065" rot="R90">
 <attribute name="SPICEPREFIX" value="C" x="8.255" y="12.065" size="1.778" layer="27" rot="R90" display="off"/>
@@
 <attribute name="SPICEPREFIX" value="C" x="71.12" y="29.21" size="1.778" layer="27" display="off"/>
 </element>
+<element name="IC4" library="adafruit" package="HTSSOP20DAP" value="TLC59711" x="54.61" y="40.64"/>
 </elements>
 <signals>
@@
 <wire x1="10.47" y1="19.9958" x2="10.4902" y2="19.9756" width="0.4064" layer="1"/>
 <wire x1="10.4902" y1="19.9756" x2="11.1252" y2="19.9756" width="0.4064" layer="1"/>
-<wire x1="11.1252" y1="19.9756" x2="15.7114" y2="19.9756" width="0.4064" layer="1"/>
-<wire x1="15.7114" y1="19.9756" x2="15.748" y2="19.939" width="0.4064" layer="1"/>
+<wire x1="11.1252" y1="19.9756" x2="13.1714" y2="19.9756" width="0.4064" layer="1"/>
 <wire x1="11.12" y1="18.6644" x2="11.12" y2="19.9704" width="0.4064" layer="1"/>
 <wire x1="11.12" y1="19.9704" x2="11.1252" y2="19.9756" width="0.4064" layer="1"/>
@@
 <wire x1="5.52" y1="35.755" x2="3.8575" y2="35.755" width="1.016" layer="1"/>
 <wire x1="6.9206" y1="34.3544" x2="5.52" y2="35.755" width="1.016" layer="1"/>
+<contactref element="IC4" pad="2"/>
+<via x="13.1714" y="19.9756" extent="1-16" drill="0.35"/>
+<wire x1="13.1714" y1="19.9756" x2="14.2494" y2="18.8976" width="0.4064" layer="16"/>
+<wire x1="14.2494" y1="18.8976" x2="14.2494" y2="13.4366" width="0.4064" layer="16"/>
+<wire x1="14.2494" y1="13.4366" x2="15.748" y2="11.938" width="0.4064" layer="16"/>
+<wire x1="15.748" y1="11.938" x2="15.748" y2="10.541" width="0.4064" layer="16"/>
 <wire x1="104.9808" y1="4.7973" x2="103.8606" y2="20.0914" width="0" layer="19" extent="1-1"/>
 <wire x1="76.7875" y1="20.665" x2="103.8606" y2="20.0914" width="0" layer="19" extent="1-1"/>
@@
 <wire x1="45.5398" y1="32.9184" x2="42.4942" y2="28.2672" width="0" layer="19" extent="1-1"/>
 <wire x1="47.9582" y1="37.465" x2="48.2752" y2="34.0692" width="0" layer="19" extent="1-1"/>
+<wire x1="52.335" y1="37.84" x2="50.0126" y2="38.2494" width="0" layer="19" extent="1-1"/>
 <wire x1="42.6578" y1="39.4836" x2="45.8778" y2="38.2636" width="0" layer="19" extent="1-1"/>
 <wire x1="42.6578" y1="40.4836" x2="42.6578" y2="39.4836" width="0" layer="19" extent="1-1"/>
@@
 <wire x1="30.1858" y1="32.771" x2="32.286390625" y2="36.8251125" width="0" layer="19" extent="1-1"/>
 <wire x1="27.2034" y1="35.013" x2="30.1858" y2="32.771" width="0" layer="19" extent="1-1"/>
-<wire x1="31.242" y1="19.939" x2="34.6858" y2="22.1848" width="0" layer="19" extent="1-1"/>
 <wire x1="48.3108" y1="46.1518" x2="45.8778" y2="42.2036" width="0" layer="19" extent="1-1"/>
-<wire x1="28.067" y1="15.872" x2="31.242" y2="19.939" width="0" layer="19" extent="1-1"/>
-<wire x1="25.273" y1="15.8974" x2="28.067" y2="15.872" width="0" layer="19" extent="1-1"/>
 <wire x1="53.3908" y1="48.6918" x2="48.3108" y2="46.1518" width="0" layer="19" extent="1-1"/>
 <wire x1="58.4708" y1="48.6918" x2="53.3908" y2="48.6918" width="0" layer="19" extent="1-1"/>
 <wire x1="65.725" y1="35.39" x2="62.015" y2="31.115" width="0" layer="19" extent="1-1"/>
+<wire x1="58.105" y1="38.565" x2="52.335" y2="37.84" width="0" layer="19" extent="1-1"/>
 <wire x1="68.5292" y1="40.9448" x2="64.92" y2="36.195" width="0" layer="19" extent="1-1"/>
 <wire x1="66.0908" y1="46.1518" x2="69.5706" y2="47.8562" width="0" layer="19" extent="1-1"/>
 <wire x1="72.52" y1="37.465" x2="68.5292" y2="40.9448" width="0" layer="19" extent="1-1"/>
 <wire x1="24.7396" y1="22.5014" x2="27.9858" y2="27.571" width="0" layer="19" extent="1-1"/>
-<wire x1="33.5788" y1="12.612" x2="28.067" y2="15.872" width="0" layer="19" extent="1-1"/>
+<wire x1="25.273" y1="15.8974" x2="24.7396" y2="22.5014" width="0" layer="19" extent="1-1"/>
+<wire x1="28.067" y1="15.872" x2="25.273" y2="15.8974" width="0" layer="19" extent="1-1"/>
+<wire x1="31.242" y1="10.541" x2="28.067" y2="15.872" width="0" layer="19" extent="1-1"/>
+<wire x1="33.5788" y1="12.612" x2="31.242" y2="10.541" width="0" layer="19" extent="1-1"/>
 <wire x1="20.6218" y1="28.0162" x2="24.7396" y2="22.5014" width="0" layer="19" extent="1-1"/>
 <wire x1="17.61" y1="28.575" x2="20.6218" y2="28.0162" width="0" layer="19" extent="1-1"/>
 <wire x1="18.2148" y1="24.765" x2="17.61" y2="28.575" width="0" layer="19" extent="1-1"/>
-<wire x1="15.748" y1="19.939" x2="18.2148" y2="24.765" width="0" layer="19" extent="1-1"/>
+<wire x1="13.1714" y1="19.9756" x2="18.2148" y2="24.765" width="0" layer="19" extent="1-1"/>
 <wire x1="7.2136" y1="19.3836" x2="9.82" y2="20.32" width="0" layer="19" extent="1-1"/>
 <wire x1="10.03" y1="27.305" x2="6.9206" y2="26.7106" width="0" layer="19" extent="1-1"/>
 <wire x1="10.03" y1="29.845" x2="10.03" y2="27.305" width="0" layer="19" extent="1-1"/>
-<wire x1="58.105" y1="38.565" x2="64.8456" y2="36.195" width="0" layer="19" extent="1-1"/>
 <wire x1="33.0708" y1="48.6918" x2="35.43" y2="41.91" width="0" layer="19" extent="1-1"/>
 <wire x1="27.9908" y1="46.1518" x2="33.0708" y2="48.6918" width="0" layer="19" extent="1-1"/>
@@
 <wire x1="56.4358" y1="31.0896" x2="59.905" y2="34.29" width="0" layer="19" extent="1-1"/>
 <wire x1="50.9134" y1="29.3878" x2="54.003" y2="27.1526" width="0" layer="19" extent="1-1"/>
-<wire x1="31.242" y1="10.541" x2="47.1034" y2="29.3878" width="0" layer="19" extent="1-1"/>
+<wire x1="31.242" y1="19.939" x2="47.1034" y2="29.3878" width="0" layer="19" extent="1-1"/>
 <wire x1="21.6688" y1="41.2496" x2="47.1034" y2="31.8634" width="0" layer="19" extent="1-1"/>
 <wire x1="13.335" y1="38.27" x2="19.05" y2="44.5034" width="0" layer="19" extent="1-1"/>
@@
 <wire x1="8.89" y1="45.2952" x2="8.89" y2="45.575" width="1.016" layer="1"/>
 <wire x1="7.4098" y1="43.815" x2="8.89" y2="45.2952" width="1.27" layer="1"/>
-<wire x1="15.748" y1="10.541" x2="15.748" y2="15.367" width="1.778" layer="1"/>
 <wire x1="14.853" y1="16.262" x2="12.065" y2="16.262" width="1.778" layer="1"/>
-<wire x1="15.748" y1="15.367" x2="14.853" y2="16.262" width="1.778" layer="1"/>
+<wire x1="14.853" y1="16.262" x2="15.748" y2="17.272" width="1.778" layer="1"/>
 <wire x1="15.41" y1="29.525" x2="13.15" y2="29.525" width="1.016" layer="1"/>
 <wire x1="13.15" y1="29.525" x2="12.83" y2="29.845" width="1.016" layer="1"/>
@@
 <wire x1="43.3324" y1="15.7226" x2="41.91" y2="17.145" width="0.6096" layer="1"/>
 <wire x1="41.91" y1="17.145" x2="41.91" y2="19.05" width="0.6096" layer="1"/>
+<wire x1="15.748" y1="17.272" x2="15.748" y2="19.939" width="1.778" layer="1"/>
 <wire x1="61.8464" y1="15.7226" x2="72.7022" y2="41.8338" width="0" layer="19" extent="1-1"/>
 <wire x1="44.803" y1="15.7226" x2="59.0804" y2="11.0998" width="0" layer="19" extent="1-1"/>
-<wire x1="15.748" y1="15.367" x2="40.64" y2="20.32" width="0" layer="19" extent="1-1"/>
-<wire x1="13.15" y1="29.525" x2="10.47" y2="18.6644" width="0" layer="19" extent="1-1"/>
+<wire x1="15.748" y1="19.939" x2="40.64" y2="20.8" width="0" layer="19" extent="1-1"/>
+<wire x1="15.41" y1="29.525" x2="15.748" y2="19.939" width="0" layer="19" extent="1-1"/>
 <wire x1="11.7068" y1="44.0944" x2="12.83" y2="29.845" width="0" layer="19" extent="1-1"/>
 </signal>
@@
 <wire x1="48.1076" y1="14.7828" x2="47.43" y2="14.1052" width="0.8128" layer="16"/>
 </signal>
+<signal name="VCC">
+<contactref element="IC4" pad="19"/>
+</signal>
 </signals>
