File: pcb/smd/zeta2/zeta2rework_lw_v6.sch (EAGLE design)
At the start: 104 parts, among them IC1 MAX6520, IC2 L293DD, IC3 L293DD, Q12 8MHz, U1 MPU-6050, U2 INA219, U5 DS18B20U+

Commit message: finished pcb
Parts:
- added IC4: TLC59711, adafruit:TLC59711
Changed lines of the file:
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@@
 <part name="+3V1" library="supply1" library_urn="urn:adsk.eagle:library:371" deviceset="+3V3" device=""/>
 <part name="C11" library="rcl" library_urn="urn:adsk.eagle:library:334" deviceset="C-EU" device="C1206" package3d_urn="urn:adsk.eagle:package:23618/2" value="0.1µF"/>
+<part name="IC4" library="adafruit" deviceset="TLC59711" device=""/>
 </parts>
 <sheets>
@@
 <instance part="+3V1" gate="G$1" x="86.36" y="-10.16"/>
 <instance part="C11" gate="G$1" x="91.44" y="7.62"/>
+<instance part="IC4" gate="G$1" x="-81.28" y="33.02"/>
 </instances>
 <busses>
