File: pcb/smd/zeta2/zeta2rework_lw_v23_fixes.brd (EAGLE design)
At the start: 81 x 45.7 mm, 81 parts, among them U5 DS18B20U+

Commit message: version 3 of pcb should be finihsed now
Parts:
- removed BOOTCONFIG: (no value), special:EDG-02
- removed R11, R15: 132k, rcl:R0603
- added R1, R2: 10k, rcl:R0603
- C1: value 10nF -> 100nF
- C20: value 0.1µF -> 10nf
- moved C1 73.8 mm to (-8.89, -14.0), turned to 0 degrees
- moved C39 11.7 mm to (35.6, 21.0), turned to 180 degrees
- moved C18 7.18 mm to (44.5, 34.3), turned to 270 degrees
- moved C20 5.24 mm to (40.6, 41.9)
- moved C21 2.54 mm to (40.6, 38.7), turned to 180 degrees
- moved C38 1.88 mm to (40.0, 32.4), turned to 90 degrees
- moved C40 1.80 mm to (29.1, 37.1)
- moved R25 0.64 mm to (40.9, 26.4)
- moved C3 0.63 mm to (40.6, 22.9)
- moved R30 0.22 mm to (27.1, 34.3)
Connections:
- removed net BOOT0: BOOTCONFIG.2, R15.2, STM32F103CB.44
- removed net BOOT1: BOOTCONFIG.1, R11.2, STM32F103CB.20
- removed net BOOT2: RPI_ZERO.29
- removed net BOOT3: RPI_ZERO.27
- new net N$5: R1.1, STM32F103CB.44
- net +3V3: now also R2.2; no longer BOOTCONFIG.3, BOOTCONFIG.4, C1.1
- net GND: now also R1.2; no longer R11.1, R15.1
- net NRST: now also C1.1, R2.1
Routing:
- net BOOT0: track 25.5 -> 0.00 mm
- net GND: track 600.0 -> 623.6 mm
- net BOOT1: track 16.0 -> 0.00 mm
- net +3V3: track 200.1 -> 204.9 mm
- net +8V: track 237.0 -> 238.7 mm
- net N$36: track 2.05 -> 3.67 mm
- net FRONT_LIGHT: track 65.9 -> 64.7 mm
- net SCL: track 106.9 -> 106.0 mm
- net SDA: track 94.6 -> 95.3 mm
