File: pcb/smd/zeta2/zeta2rework_lw_v23_fixes.sch (EAGLE design)
At the start: 81 parts, among them U5 DS18B20U+

Commit message: version 3 of pcb should be finihsed now
Parts:
- removed BOOTCONFIG: (no value), special:SW_DIP-2
- removed R11, R15: 132k, rcl:R-EU_R0603
- added R1, R2: 10k, rcl:R-EU_R0603
- C1: value 10nF -> 100nF
- C20: value 0.1µF -> 10nf
Connections:
- removed net BOOT0: BOOTCONFIG.2, R15.2, STM32F103CB.BOOT0
- removed net BOOT1: BOOTCONFIG.1, R11.2, STM32F103CB.PB2
- removed net BOOT2: RPI_ZERO.29
- removed net BOOT3: RPI_ZERO.27
- new net N$5: R1.1, STM32F103CB.BOOT0
- net +3V3: now also R2.2; no longer BOOTCONFIG.3, BOOTCONFIG.4, C1.1
- net GND: now also R1.2; no longer R11.1, R15.1
- net NRST: now also C1.1, R2.1
Other:
- moved on the sheet: C1, C10, C11, C18, C20, C34, C43, D1, D3, FAN, FRONTLIGHT, IRLML1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
