File: pcb/smd/zeta2/zeta2rework_lw_v24_fixes.brd (EAGLE design)
At the start: 81 x 45.7 mm, 80 parts, among them U5 DS18B20U+

Commit message: version 3 of pcb should be finihsed now
Parts:
- removed BOOTCONFIG: (no value), special:EDG-02
- removed R11, R15: 132k, rcl:R0603
- removed SCL, SDA: TPSQTP20R, testpad:TP20R
- added C1: 100nF, rcl:C1206
- added J1: B4B-ZR(LF)(SN), B4B-ZR(LF)(SN):SHDR4W50P0X150_1X4_750X350X450
- added R1, R2: 10k, rcl:R0603
- R18: value 500 -> 500R
- moved 3.3V 12.7 mm to (13.3, 31.8)
- moved GND 12.3 mm to (13.3, 35.6)
- moved R29 12.1 mm to (12.3, 30.3), turned to 0 degrees
- moved R20 8.19 mm to (15.6, 30.3), turned to 180 degrees
- moved C3 5.07 mm to (39.9, 17.9)
- moved C39 4.26 mm to (39.4, 22.9), turned to 0 degrees
- moved C40 1.63 mm to (29.2, 38.7)
- moved C12 1.27 mm to (59.1, 13.4)
- moved C36 0.63 mm to (22.0, 28.7)
- moved R18 0.55 mm to (77.5, 10.2), turned to 90 degrees
- moved Q9 0.33 mm to (77.3, 14.6), turned to 0 degrees
- moved C33 0.23 mm to (24.8, 24.1)
Connections:
- removed net BOOT0: BOOTCONFIG.2, R15.2, STM32F103CB.44
- removed net BOOT1: BOOTCONFIG.1, R11.2, STM32F103CB.20
- removed net BOOT2: RPI_ZERO.29
- removed net BOOT3: RPI_ZERO.27
- removed net N$20: Q9.2, R3.1
- new net INT_MD_1: J1.3, STM32F103CB.21
- new net INT_MD_2: J1.2, STM32F103CB.22
- new net N$5: R1.1, STM32F103CB.44
- new net N$7: FRONTLIGHT.P2, Q9.3
- net +3V3: now also R2.2; no longer BOOTCONFIG.3, BOOTCONFIG.4
- net +5V: now also J1.4, R3.1; no longer Q9.3
- net GND: now also C1.2, J1.1, Q9.2, R1.2; no longer FRONTLIGHT.P2, R11.1, R15.1
- net MPU_INT: now also STM32F103CB.41
- net NRST: now also C1.1, R2.1
- net SCL: no longer SCL.TP
- net SDA: no longer SDA.TP
Routing:
- net BOOT0: track 27.8 -> 0.00 mm
- net BOOT1: track 19.3 -> 0.00 mm
- net MPU_INT: track 0.00 -> 17.4 mm, vias 0 -> 2
- net SCL: track 106.0 -> 89.6 mm, vias 4 -> 3
- net INT_MD_2: track 0.00 -> 14.9 mm
- net INT_MD_1: track 0.00 -> 14.5 mm
- net N$20: track 10.7 -> 0.00 mm
- net +3V3: track 216.1 -> 207.8 mm
- net SDA: track 95.3 -> 87.8 mm
- net +5V: track 220.9 -> 227.2 mm
- net GND: track 634.0 -> 639.8 mm, vias 7 -> 8
- net NRST: track 30.2 -> 35.7 mm
- net N$5: track 0.00 -> 4.25 mm
- net N$7: track 0.00 -> 3.94 mm
- net +8V: track 238.7 -> 236.1 mm
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- added copper zone on layer 16, net +8V
Other:
- board text added: "5v I1 I2 GND"
- board text added: "TODO: die SDA SCL pinups vllt zum INA und PCA hoch machen"
- board text removed: "TODO: am untersten rechten (pin24) 3.3v vom stm32 fehlt der kondensator"
- board text removed: "TODO: heatsink thermal for +3v3"
