File: pcb/smd/zeta2/zeta2rework_lw_v24_fixes.sch (EAGLE design)
At the start: 80 parts, among them U5 DS18B20U+

Commit message: version 3 of pcb should be finihsed now
Parts:
- removed BOOTCONFIG: (no value), special:SW_DIP-2
- removed R11, R15: 132k, rcl:R-EU_R0603
- removed SCL, SDA: TPSQTP20R, testpad:TPSQTP20R
- added C1: 100nF, rcl:C-EUC1206
- added J1: B4B-ZR(LF)(SN), B4B-ZR(LF)(SN):B4B-ZR(LF)(SN)
- added R1, R2: 10k, rcl:R-EU_R0603
- R18: value 500 -> 500R
Connections:
- removed net BOOT0: BOOTCONFIG.2, R15.2, STM32F103CB.BOOT0
- removed net BOOT1: BOOTCONFIG.1, R11.2, STM32F103CB.PB2
- removed net BOOT2: RPI_ZERO.29
- removed net BOOT3: RPI_ZERO.27
- removed net N$20: Q9.E, R3.1
- new net INT_MD_1: J1.3, STM32F103CB.PB10
- new net INT_MD_2: J1.2, STM32F103CB.PB11
- new net N$5: R1.1, STM32F103CB.BOOT0
- new net N$7: FRONTLIGHT.2, Q9.C
- net +3V3: now also R2.2; no longer BOOTCONFIG.3, BOOTCONFIG.4
- net +5V: now also J1.4, R3.1; no longer Q9.C
- net GND: now also C1.2, J1.1, Q9.E, R1.2; no longer FRONTLIGHT.2, R11.1, R15.1
- net MPU_INT: now also STM32F103CB.PB5
- net NRST: now also C1.1, R2.1
- net SCL: no longer SCL.TP
- net SDA: no longer SDA.TP
Other:
- moved on the sheet: 3.3V, C10, C11, C12, C17, C18, C2, C20, C21, C23, C24, C3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
