File: pcb/smd/zeta2/zeta2rework_lw_v25_fixes_wompu.brd (EAGLE design)
At the start: 81 x 45.7 mm, 80 parts, among them U5 DS18B20U+

Commit message: version 3 of pcb should be finihsed now
Parts:
- removed BOOTCONFIG: (no value), special:EDG-02
- removed C11, C18, C21: 0.1µF, rcl:C1206
- removed C20: 10nf, rcl:C1206
- removed IRLML1, IRLML2502: (no value), zetex:SOT-23
- removed MPU6050: MPU-6050, MPU-6050:QFN50P400X400X95-24N
- removed Q9: (no value), semicon-smd-ipc:SOT23
- removed R11, R15: 132k, rcl:R0603
- removed R18: 500, rcl:R0603
- removed SCL, SDA: TPSQTP20R, testpad:TP20R
- added 1.8V_CONV: MCP1700T-1802E/TT, MCP1700T-2102E_TT:SOT95P237X112-3N
- added 1K: 22R, rcl:R0603
- added C1: 100nF, rcl:C1206
- added C14: 1µF, rcl:C1206
- added C6, C7, C8: 0.1nF, rcl:C1206
- added J1: B4B-ZR(LF)(SN), B4B-ZR(LF)(SN):SHDR4W50P0X150_1X4_750X350X450
- added M1, M2, M3: IRLML2502, IRLML2502TRPBF:SOT23
- added R1, R2: 10k, rcl:R0603
- added U3: ICM-20948, ICM-20948:QFN40P300X300X105-25N
- C10, C12, C3, C34, C43: device rcl:UD-4X5,8_NICHICON -> rcl:UD-5X5,8_NICHICON
- C17: value 2,2nF -> 1µF
- C36, C37: value 22pf -> 7pf
- R10, R12, R14, R4, R7, R8: value 100k -> 10k
- R3: value 220R -> 0R
- moved 3.3V 12.7 mm to (13.3, 31.8)
- moved GND 12.3 mm to (13.3, 35.6)
- moved R29 12.1 mm to (12.3, 30.3), turned to 0 degrees
- moved C17 11.3 mm to (41.9, 37.5), turned to 90 degrees
- moved R20 8.19 mm to (15.6, 30.3), turned to 180 degrees
- moved C3 4.76 mm to (39.9, 18.2)
- moved R12 4.49 mm to (48.3, 31.1), turned to 90 degrees
- moved C39 4.26 mm to (39.4, 22.9), turned to 0 degrees
- moved R14 3.49 mm to (52.3, 31.1), turned to 90 degrees
- moved R8 2.36 mm to (50.3, 31.1), turned to 90 degrees
- moved C12 0.72 mm to (58.9, 12.8)
- moved C10 0.64 mm to (71.1, 47.3)
- moved MOTOR_R_F 0.64 mm to (52.7, 11.4)
- moved C36 0.63 mm to (22.0, 28.7)
- moved MOTOR_R_B 0.63 mm to (45.7, 11.4)
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- renumbered 3.3V_CONF to 3.3V_CONV
Connections:
- removed net BOOT0: BOOTCONFIG.2, R15.2, STM32F103CB.44
- removed net BOOT1: BOOTCONFIG.1, R11.2, STM32F103CB.20
- removed net BOOT2: RPI_ZERO.29
- removed net BOOT3: RPI_ZERO.27
- removed net MPU_INT: MPU6050.12
- removed net N$19: Q9.1, R18.2
- removed net N$20: Q9.2, R3.1
- removed net N$34: C17.1, MPU6050.20
- removed net N$36: C21.1, MPU6050.10
- new net +1.8V: 1.8V_CONV.2, C14.1, C8.1, U3.8
- new net INT_MD_1: J1.3, STM32F103CB.21
- new net INT_MD_2: J1.2, STM32F103CB.22
- new net N$10: 1K.2, M3.1
- new net N$5: R1.1, STM32F103CB.44
- new net N$8: C7.1, U3.10
- new net N$9: FRONTLIGHT.P2, M3.3
- net +3V3: now also 1.8V_CONV.3, C17.1, C6.1, R2.2, U3.13; no longer BOOTCONFIG.3, BOOTCONFIG.4, C18.1, C20.1, MPU6050.13, MPU6050.8
- net +5V: now also 3.3V_CONV.3, C15.1, J1.4, R3.1; no longer C11.1, Q9.3
- net +8V: no longer 3.3V_CONV.3, C15.1
- net FRONT_LIGHT: now also 1K.1; no longer R18.1
- net GND: now also 1.8V_CONV.1, C1.2, C14.2, C6.2, C7.2, C8.2, J1.1, M1.2, M2.2, M3.2, R1.2, U3.18; no longer C11.2, C18.2, C20.2, C21.2, FRONTLIGHT.P2, IRLML1.2, IRLML2502.2, MPU6050.1, MPU6050.11, MPU6050.18, MPU6050.9, R11.1, R15.1
- net N$37: now also M2.1; no longer IRLML2502.3
- net N$38: now also M1.1; no longer IRLML1.3
- net N$39: now also M1.3; no longer IRLML1.1
- net N$55: now also M2.3; no longer IRLML2502.1
- net NRST: now also C1.1, R2.1
- net SCL: now also U3.23; no longer MPU6050.23, SCL.TP
- net SDA: now also U3.24; no longer MPU6050.24, SDA.TP
Routing:
- net BOOT0: track 27.8 -> 0.00 mm
- net +3V3: track 216.1 -> 192.8 mm
- net BOOT1: track 19.3 -> 0.00 mm
- net GND: track 634.0 -> 616.7 mm
- net SCL: track 106.0 -> 89.8 mm, vias 4 -> 3
- net INT_MD_2: track 0.00 -> 14.9 mm
- net INT_MD_1: track 0.00 -> 14.5 mm
- net +1.8V: track 0.00 -> 14.4 mm
- net N$20: track 10.7 -> 0.00 mm
- net +5V: track 220.9 -> 230.1 mm, vias 1 -> 2
- net NRST: track 30.2 -> 38.4 mm
- net SDA: track 95.3 -> 87.8 mm
- net +8V: track 238.7 -> 232.8 mm
- net N$8: track 0.00 -> 4.53 mm
- net N$5: track 0.00 -> 4.25 mm
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- added copper zone on layer 16, net +8V
Other:
- board text added: "5v I1 I2 GND"
- board text added: "TODO: 2n2222 resistors"
- board text added: "TODO: STM32 crystal and capacitro checken - typical applciation im datasheet"
- board text added: "TODO: i2c fast mode check, stm32 werte richtig? ncohmal im datasheet schauen bzgl typical application for clocksxspeed, crystal vals are vermutlkich falsch"
- board text removed: "TODO: am untersten rechten (pin24) 3.3v vom stm32 fehlt der kondensator"
- board text removed: "TODO: heatsink thermal for +3v3"
