File: pcb/smd/zeta2/zeta2rework_lw_v25_fixes_wompu.sch (EAGLE design)
At the start: 80 parts, among them U5 DS18B20U+

Commit message: version 3 of pcb should be finihsed now
Parts:
- removed 3.3V_CONF: NCP1117LPST33T3G, NCP1117LPST33T3G:NCP1117LPST33T3G
- removed BOOTCONFIG: (no value), special:SW_DIP-2
- removed C11, C18, C21: 0.1µF, rcl:C-EUC1206
- removed C20: 10nf, rcl:C-EUC1206
- removed IRLML1, IRLML2502: (no value), zetex:NMOSSOT23
- removed MPU6050: MPU-6050, MPU-6050:MPU-6050
- removed Q9: (no value), semicon-smd-ipc:NPN-TRANSISTOR_SOT23
- removed R11, R15: 132k, rcl:R-EU_R0603
- removed R18: 500, rcl:R-EU_R0603
- removed SCL, SDA: TPSQTP20R, testpad:TPSQTP20R
- added 1.8V_CONV: MCP1700T-1802E/TT, MCP1700T-2102E_TT:MCP1700T-2102E/TT
- added 1K: 22R, rcl:R-EU_R0603
- added 3.3V_CONV: NCP1117LPST33T3G, NCP1117LPST33T3G:NCP1117LPST33T3G
- added C1: 100nF, rcl:C-EUC1206
- added C14: 1µF, rcl:C-EUC1206
- added C6, C7, C8: 0.1nF, rcl:C-EUC1206
- added J1: B4B-ZR(LF)(SN), B4B-ZR(LF)(SN):B4B-ZR(LF)(SN)
- added M1, M2, M3: IRLML2502, IRLML2502TRPBF:IRLML2502TRPBF
- added R1, R2: 10k, rcl:R-EU_R0603
- added U3: ICM-20948, ICM-20948:ICM-20948
- C10, C12, C3, C34, C43: device rcl:CPOL-EUUD-4X5,8 -> rcl:CPOL-EUUD-5X5,8
- C17: value 2,2nF -> 1µF
- C36, C37: value 22pf -> 7pf
- R10, R12, R14, R4, R7, R8: value 100k -> 10k
- R3: value 220R -> 0R
Connections:
- removed net BOOT0: BOOTCONFIG.2, R15.2, STM32F103CB.BOOT0
- removed net BOOT1: BOOTCONFIG.1, R11.2, STM32F103CB.PB2
- removed net BOOT2: RPI_ZERO.29
- removed net BOOT3: RPI_ZERO.27
- removed net MPU_INT: MPU6050.INT
- removed net N$19: Q9.B, R18.2
- removed net N$20: Q9.E, R3.1
- removed net N$34: C17.1, MPU6050.CPOUT
- removed net N$36: C21.1, MPU6050.REGOUT
- new net +1.8V: 1.8V_CONV.VOUT, C14.1, C8.1, U3.VDDIO
- new net INT_MD_1: J1.3, STM32F103CB.PB10
- new net INT_MD_2: J1.2, STM32F103CB.PB11
- new net N$10: 1K.2, M3.G
- new net N$5: R1.1, STM32F103CB.BOOT0
- new net N$8: C7.1, U3.REGOUT
- new net N$9: FRONTLIGHT.2, M3.D
- net +3V3: now also 1.8V_CONV.VIN, 3.3V_CONV.OUTPUT, C17.1, C6.1, R2.2, U3.VDD; no longer 3.3V_CONF.OUTPUT, BOOTCONFIG.3, BOOTCONFIG.4, C18.1, C20.1, MPU6050.VDD, MPU6050.VLOGIC
- net +5V: now also 3.3V_CONV.INPUT, C15.1, J1.4, R3.1; no longer C11.1, Q9.C
- net +8V: no longer 3.3V_CONF.INPUT, C15.1
- net FRONT_LIGHT: now also 1K.1; no longer R18.1
- net GND: now also 1.8V_CONV.GND, 3.3V_CONV.GND, C1.2, C14.2, C6.2, C7.2, C8.2, J1.1, M1.S, M2.S, M3.S, R1.2, U3.GND; no longer 3.3V_CONF.GND, C11.2, C18.2, C20.2, C21.2, FRONTLIGHT.2, IRLML1.S, IRLML2502.S, MPU6050.AD0, MPU6050.CLKIN, MPU6050.FSYNC, MPU6050.GND, R11.1, R15.1
- net N$37: now also M2.G; no longer IRLML2502.G
- net N$38: now also M1.G; no longer IRLML1.G
- net N$39: now also M1.D; no longer IRLML1.D
- net N$55: now also M2.D; no longer IRLML2502.D
- net NRST: now also C1.1, R2.1
- net SCL: now also U3.SCL/SCLK; no longer MPU6050.SCL, SCL.TP
- net SDA: now also U3.SDA/SDI; no longer MPU6050.SDA, SDA.TP
Other:
- moved on the sheet: 3.3V, 5V_CONV, C10, C12, C13, C15, C16, C17, C2, C23, C24, C27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
