File: pcb/smd/zeta2/zeta2rework_lw_v27_rework.brd (EAGLE design)
At the start: 81 x 50.2 mm, 83 parts, among them IC1 DRV8844PWPR, IC2 DRV8844PWPR, J1 B4B-ZR(LF)(SN), M1 IRLML2502, M2 IRLML2502, M3 IRLML2502, U1 STM32F427VGT7, U3 ICM-20948, U5 DS18B20U+

Commit message: using stm32f4, fixed pin settings, added cubemx
Parts:
- removed C1: 100nF, rcl:C1206
- removed C33, C38, C39, C40: 10nF, rcl:C1206
- removed C36, C37: 22pf, rcl:C1206
- removed J1: B4B-ZR(LF)(SN), B4B-ZR(LF)(SN):SHDR4W50P0X150_1X4_750X350X450
- removed KX-9A: 8Mhz, crystal-geyer_V1_0:5.0X3.2_KX-9A
- removed R20, R29: 10k, rcl:R0603
- removed R30: 100k, rcl:R0603
- removed STM32F103CB: STM32F103CB, STM32F103C8T6:LQFP48_7X7MM_0.5MMPP
- added C11, C12: 0pf, rcl:C1206
- added C28, C35, C41, C42, C44, C45, C46, C47, C49, C50: 100nF, rcl:C1206
- added C29, C32: 2.2µf Low ESR < 2ohm, rcl:C1206
- added C48: 4.7µf, rcl:SMC_P
- added C51: 1µf, rcl:C1206
- added R10, R4, R7, R8: 10k, rcl:R0603
- added R15: 0k, rcl:R0603
- added X1: 25mhz, crystal-geyer_V1_0:5.0X3.2_KX-9A
- C6: device rcl:C1206 -> rcl:C0603
- U1: value STM32F427VGT7 -> STM32F427VI
- moved R1 412.3 mm to (-40.6, -363.9), turned to 0 degrees
- moved R2 400.5 mm to (-40.6, -368.9), turned to 0 degrees
Connections:
- removed net FRONT_LIGHT: R6.1, STM32F103CB.27
- removed net INT_MD_1: J1.3, STM32F103CB.21
- removed net INT_MD_2: J1.2, STM32F103CB.22
- removed net M_DIR_L_1: STM32F103CB.39
- removed net M_DIR_L_2: STM32F103CB.38
- removed net M_DIR_R_1: STM32F103CB.14
- removed net M_DIR_R_2: STM32F103CB.15
- removed net N$46: C36.2, KX-9A.1, STM32F103CB.6
- removed net N$47: C37.2, KX-9A.3, STM32F103CB.5
- removed net N$49: R30.1, STM32F103CB.2
- removed net N$5: R1.1, STM32F103CB.44
- removed net PWM_M_EN_L: STM32F103CB.16
- removed net PWM_M_EN_R: STM32F103CB.17
- removed net SCL: I2C.1, INA219.5, PCA9533.6, R29.2, STM32F103CB.42, U3.23
- removed net SDA: I2C.2, INA219.6, PCA9533.7, R20.2, STM32F103CB.43, U3.24
- removed net U1_RX: LDIAR.P1, STM32F103CB.31
- removed net U1_TX: LDIAR.P2, STM32F103CB.30
- removed net USART2_RX: RPI_ZERO.34, STM32F103CB.13
- removed net USART2_TX: RPI_ZERO.32, STM32F103CB.12
- removed net USB_DM: STM32F103CB.32
- removed net USB_DP: STM32F103CB.33
- removed net VBAT: U1.6
- removed net VCAP_1: U1.49
- removed net VCAP_2: U1.73
- removed net VDD: U1.100, U1.11, U1.19, U1.28, U1.50, U1.75
- removed net VDDA: U1.22
- removed net VREF+: U1.21
- removed net VSS: U1.10, U1.27, U1.74, U1.99
- removed net VSSA: U1.20
- new net I2C1_SCL: INA219.5, PCA9533.6, R1.2, U1.92, U3.23
- new net I2C1_SDA: INA219.6, PCA9533.7, R2.2, U1.93, U3.24
- new net I2C3_SCL: I2C.1, R4.2, U1.67
- new net I2C3_SDA: I2C.2, R10.2, U1.66
- new net N$13: C11.2, U1.13, X1.1
- new net N$14: C12.2, R15.2, X1.3
- new net N$16: R7.1, U1.94
- new net N$36: C29.2, U1.49
- new net N$44: R15.1, U1.12
- new net N$45: C32.2, U1.73
- new net PWM1: U1.47
- new net PWM2: U1.48
- new net PWM3: U1.35
- new net PWM4: U1.36
- new net PWM_LIGHT: R6.1, U1.40
- new net UART2_RX: U1.26
- new net UART2_TX: U1.25
- new net UART3_RX: U1.56
- new net UART3_TX: U1.55
- new net UART4_RX: RPI_ZERO.34, U1.79
- new net UART4_TX: RPI_ZERO.32, U1.78
- new net USART3_RX: LDIAR.P1
- new net USART3_TX: LDIAR.P2
- new net USB_OTG_DM: U1.70
- new net USB_OTG_DP: U1.71
- new net USB_OTG_ID: U1.69
- new net USB_OTG_VBUS: U1.68
- net +3V3: now also C35.1, C41.1, C42.1, C44.1, C45.1, C46.1, C47.1, C48.+, C49.1, C50.1, C51.1, R1.1, R10.1, R2.1, R4.1, R8.2, U1.100, U1.11, U1.19, U1.21, U1.22, U1.28, U1.50, U1.6, U1.75; no longer C33.1, C38.1, C39.1, C40.1, R2.2, R20.1, R29.1, STM32F103CB.1, STM32F103CB.24, STM32F103CB.36, STM32F103CB.48, STM32F103CB.9
- net +5V: no longer J1.4
- net BAT_LVL: now also U1.15; no longer STM32F103CB.10
- net DEC_LB_1: now also U1.31
- net DEC_LB_2: now also U1.32
- net DEC_LF_1: now also U1.23
- net DEC_LF_2: now also U1.24
- net DEC_RB_1: now also U1.63
- net DEC_RB_2: now also U1.64
- net DEC_RF_1: now also U1.59
- net DEC_RF_2: now also U1.60
- net GND: now also C11.1, C12.1, C28.2, C29.1, C32.1, C35.2, C41.2, C42.2, C44.2, C45.2, C46.2, C47.2, C48.-, C49.2, C50.2, C51.2, R7.2, U1.10, U1.20, U1.27, U1.74, U1.99; no longer C1.2, C33.2, C36.1, C37.1, C38.2, C39.2, C40.2, J1.1, R1.2, R30.2, STM32F103CB.23, STM32F103CB.35, STM32F103CB.47, STM32F103CB.8
- net LIDAR_POS_INT: now also U1.81; no longer STM32F103CB.25
- net M_LB_IN1: now also U1.84
- net M_LB_IN2: now also U1.85
- net M_LF_IN1: now also U1.82
- net M_LF_IN2: now also U1.83
- net M_PWM_LB: now also U1.45
- net M_PWM_LF: now also U1.44
- net M_PWM_RB: now also U1.5
- net M_PWM_RF: now also U1.4
- net M_RB_IN1: now also U1.88
- net M_RB_IN2: now also U1.89
- net M_RF_IN1: now also U1.86
- net M_RF_IN2: now also U1.87
- net M_SLEEP: now also U1.90
- net NRST: now also C28.1, R8.1, U1.14; no longer C1.1, R2.1, STM32F103CB.7
- net PWM_FAN: now also U1.96; no longer STM32F103CB.18
- net PWM_LIDAR: now also U1.95; no longer STM32F103CB.19
- net SWCLK: now also U1.76; no longer STM32F103CB.37
- net SWDIO: now also U1.72; no longer STM32F103CB.34
- net TEMPERATURE: now also U1.42; no longer STM32F103CB.28
Routing:
- net SDA: track 90.6 -> 0.00 mm, vias 3 -> 0
- net SCL: track 84.6 -> 0.00 mm, vias 3 -> 0
- net FRONT_LIGHT: track 67.7 -> 0.00 mm, vias 2 -> 0
- net PWM_LIGHT: track 0.00 -> 66.4 mm, vias 0 -> 2
- net M_DIR_R_1: track 46.6 -> 0.00 mm, vias 2 -> 0
- net GND: track 524.5 -> 479.6 mm
- net M_DIR_R_2: track 44.3 -> 0.00 mm, vias 2 -> 0
- net PWM_M_EN_R: track 44.1 -> 0.00 mm, vias 2 -> 0
- net U1_RX: track 43.4 -> 0.00 mm, vias 1 -> 0
- net U1_TX: track 42.8 -> 0.00 mm, vias 1 -> 0
- net USART3_RX: track 0.00 -> 42.2 mm, vias 0 -> 1
- net USART3_TX: track 0.00 -> 41.4 mm, vias 0 -> 1
- net PWM_M_EN_L: track 41.0 -> 0.00 mm, vias 2 -> 0
- net +3V3: track 175.0 -> 138.5 mm, vias 10 -> 8
- net M_DIR_L_1: track 35.0 -> 0.00 mm, vias 2 -> 0
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
Commit message: added usb
Parts:
- added D2: BAT60JFILM, BAT60JFILM:SOD2513X117N
- added J1: UJ2-MIBH2-4-SMT-TR, UJ2-MIBH2-4-SMT-TR:CUI_UJ2-MIBH2-4-SMT-TR
- added R12: 1k5, rcl:R0603
- added R14, R18: 22r, rcl:R0603
- added R16: 100k, rcl:R0603
- added R19: 100r, rcl:R0603
- moved U1 3.81 mm to (31.1, 29.8)
Connections:
- new net N$15: D2.2, J1.1
- new net N$17: J1.4, R16.2
- new net N$34: J1.2, R14.2
- new net N$40: J1.SH1, J1.SH2, J1.SH3, J1.SH4, J1.SH5, R19.2
- new net N$5: J1.3, R12.1, R18.2
- net +3V3: now also R12.2
- net +5V: now also D2.1
- net GND: now also J1.5, R19.1
- net USB_OTG_DM: now also R14.1
- net USB_OTG_DP: now also R18.1
- net USB_OTG_ID: now also R16.1
Routing:
- net +5V: track 217.5 -> 213.5 mm
- net GND: track 479.6 -> 478.1 mm

Commit message: working on new pcb layout
Parts:
- added R20: 100k, rcl:R0603
- R11, R13, R9: value 10k -> 100k
Connections:
- new net NFAULT: IC1.18, IC2.18, R20.1, U1.80
- net +3V3: now also R20.2
Changed lines of the file:
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@@
 <attribute name="SPICEPREFIX" value="C" x="-49.53" y="-85.725" size="1.778" layer="27" display="off"/>
 </element>
-<element name="R9" library="rcl" library_urn="urn:adsk.eagle:library:334" package="R0603" package3d_urn="urn:adsk.eagle:package:23555/2" value="10k" x="-40.64" y="-80.645">
+<element name="R9" library="rcl" library_urn="urn:adsk.eagle:library:334" package="R0603" package3d_urn="urn:adsk.eagle:package:23555/2" value="100k" x="-40.64" y="-80.645">
 <attribute name="SPICEPREFIX" value="R" x="-40.64" y="-80.645" size="1.778" layer="27" display="off"/>
 </element>
-<element name="R11" library="rcl" library_urn="urn:adsk.eagle:library:334" package="R0603" package3d_urn="urn:adsk.eagle:package:23555/2" value="10k" x="-40.64" y="-85.725">
+<element name="R11" library="rcl" library_urn="urn:adsk.eagle:library:334" package="R0603" package3d_urn="urn:adsk.eagle:package:23555/2" value="100k" x="-40.64" y="-85.725">
 <attribute name="SPICEPREFIX" value="R" x="-40.64" y="-85.725" size="1.778" layer="27" display="off"/>
 </element>
-<element name="R13" library="rcl" library_urn="urn:adsk.eagle:library:334" package="R0603" package3d_urn="urn:adsk.eagle:package:23555/2" value="10k" x="-40.64" y="-90.805">
+<element name="R13" library="rcl" library_urn="urn:adsk.eagle:library:334" package="R0603" package3d_urn="urn:adsk.eagle:package:23555/2" value="100k" x="-40.64" y="-90.805">
 <attribute name="SPICEPREFIX" value="R" x="-40.64" y="-90.805" size="1.778" layer="27" display="off"/>
 </element>
@@
 <element name="R19" library="rcl" library_urn="urn:adsk.eagle:library:334" package="R0603" package3d_urn="urn:adsk.eagle:package:23555/2" value="100r" x="-41.91" y="-421.64">
 <attribute name="SPICEPREFIX" value="R" x="-41.91" y="-421.64" size="1.778" layer="27" display="off"/>
+</element>
+<element name="R20" library="rcl" library_urn="urn:adsk.eagle:library:334" package="R0603" package3d_urn="urn:adsk.eagle:package:23555/2" value="100k" x="-41.91" y="-426.72">
+<attribute name="SPICEPREFIX" value="R" x="-41.91" y="-426.72" size="1.778" layer="27" display="off"/>
 </element>
 </elements>
@@
 <contactref element="R4" pad="1"/>
 <contactref element="R12" pad="2"/>
+<contactref element="R20" pad="2"/>
+<wire x1="-39.79" y1="-398.78" x2="-41.06" y2="-426.72" width="0" layer="19" extent="1-1"/>
+<wire x1="-41.49" y1="-379.095" x2="-39.79" y2="-398.78" width="0" layer="19" extent="1-1"/>
+<wire x1="-41.49" y1="-374.015" x2="-41.49" y2="-379.095" width="0" layer="19" extent="1-1"/>
+<wire x1="-41.49" y1="-368.935" x2="-41.49" y2="-374.015" width="0" layer="19" extent="1-1"/>
+<wire x1="-41.49" y1="-363.855" x2="-41.49" y2="-368.935" width="0" layer="19" extent="1-1"/>
+<wire x1="-41.405" y1="-358.14" x2="-41.49" y2="-363.855" width="0" layer="19" extent="1-1"/>
+<wire x1="-41.405" y1="-351.79" x2="-41.405" y2="-358.14" width="0" layer="19" extent="1-1"/>
+<wire x1="-41.405" y1="-345.44" x2="-41.405" y2="-351.79" width="0" layer="19" extent="1-1"/>
+<wire x1="-39.675" y1="-339.09" x2="-41.405" y2="-345.44" width="0" layer="19" extent="1-1"/>
+<wire x1="-41.405" y1="-326.39" x2="-39.675" y2="-339.09" width="0" layer="19" extent="1-1"/>
+<wire x1="-41.405" y1="-320.04" x2="-41.405" y2="-326.39" width="0" layer="19" extent="1-1"/>
+<wire x1="-41.405" y1="-313.69" x2="-41.405" y2="-320.04" width="0" layer="19" extent="1-1"/>
+<wire x1="-41.405" y1="-307.34" x2="-41.405" y2="-313.69" width="0" layer="19" extent="1-1"/>
+<wire x1="-41.405" y1="-300.99" x2="-41.405" y2="-307.34" width="0" layer="19" extent="1-1"/>
+<wire x1="-41.405" y1="-294.64" x2="-41.405" y2="-300.99" width="0" layer="19" extent="1-1"/>
+<wire x1="-41.405" y1="-288.29" x2="-41.405" y2="-294.64" width="0" layer="19" extent="1-1"/>
+<wire x1="-23.915" y1="-236.855" x2="-41.405" y2="-288.29" width="0" layer="19" extent="1-1"/>
+<wire x1="-31.987" y1="-162.96" x2="-23.915" y2="-236.855" width="0" layer="19" extent="1-1"/>
 <wire x1="-37.846" y1="-147.955" x2="-31.987" y2="-162.96" width="0" layer="19" extent="1-1"/>
-<wire x1="-23.915" y1="-236.855" x2="-31.987" y2="-162.96" width="0" layer="19" extent="1-1"/>
-<wire x1="-41.405" y1="-288.29" x2="-23.915" y2="-236.855" width="0" layer="19" extent="1-1"/>
-<wire x1="-41.405" y1="-294.64" x2="-41.405" y2="-288.29" width="0" layer="19" extent="1-1"/>
-<wire x1="-41.405" y1="-300.99" x2="-41.405" y2="-294.64" width="0" layer="19" extent="1-1"/>
-<wire x1="-41.405" y1="-307.34" x2="-41.405" y2="-300.99" width="0" layer="19" extent="1-1"/>
-<wire x1="-41.405" y1="-313.69" x2="-41.405" y2="-307.34" width="0" layer="19" extent="1-1"/>
-<wire x1="-41.405" y1="-320.04" x2="-41.405" y2="-313.69" width="0" layer="19" extent="1-1"/>
-<wire x1="-41.405" y1="-326.39" x2="-41.405" y2="-320.04" width="0" layer="19" extent="1-1"/>
-<wire x1="-39.675" y1="-339.09" x2="-41.405" y2="-326.39" width="0" layer="19" extent="1-1"/>
-<wire x1="-41.405" y1="-345.44" x2="-39.675" y2="-339.09" width="0" layer="19" extent="1-1"/>
-<wire x1="-41.405" y1="-351.79" x2="-41.405" y2="-345.44" width="0" layer="19" extent="1-1"/>
-<wire x1="-41.405" y1="-358.14" x2="-41.405" y2="-351.79" width="0" layer="19" extent="1-1"/>
-<wire x1="-41.49" y1="-363.855" x2="-41.405" y2="-358.14" width="0" layer="19" extent="1-1"/>
-<wire x1="-41.49" y1="-368.935" x2="-41.49" y2="-363.855" width="0" layer="19" extent="1-1"/>
-<wire x1="-41.49" y1="-374.015" x2="-41.49" y2="-368.935" width="0" layer="19" extent="1-1"/>
-<wire x1="-41.49" y1="-379.095" x2="-41.49" y2="-374.015" width="0" layer="19" extent="1-1"/>
-<wire x1="-39.79" y1="-398.78" x2="-41.49" y2="-379.095" width="0" layer="19" extent="1-1"/>
 <wire x1="22.86" y1="15.9" x2="-37.846" y2="-147.955" width="0" layer="19" extent="1-1"/>
 <wire x1="22.86" y1="22.2" x2="22.86" y2="15.9" width="0" layer="19" extent="1-1"/>
-<wire x1="38.815" y1="35.845" x2="38.8112" y2="40.4368" width="0" layer="19" extent="1-1"/>
-<wire x1="26.115" y1="22.145" x2="26.035" y2="24.765" width="0" layer="19" extent="1-1"/>
-<wire x1="37.115" y1="22.145" x2="39.367" y2="28.702" width="0" layer="19" extent="1-1"/>
-<wire x1="23.415" y1="25.345" x2="26.115" y2="22.145" width="0" layer="19" extent="1-1"/>
+<wire x1="23.415" y1="25.345" x2="22.86" y2="24.765" width="0" layer="19" extent="1-1"/>
 <wire x1="23.415" y1="25.845" x2="23.415" y2="25.345" width="0" layer="19" extent="1-1"/>
 <wire x1="23.415" y1="26.845" x2="23.415" y2="25.845" width="0" layer="19" extent="1-1"/>
+<wire x1="38.815" y1="35.845" x2="39.919" y2="35.516" width="0" layer="19" extent="1-1"/>
+<wire x1="26.115" y1="22.145" x2="27.94" y2="22.225" width="0" layer="19" extent="1-1"/>
+<wire x1="37.115" y1="22.145" x2="38.0746" y2="20.4724" width="0" layer="19" extent="1-1"/>
 <wire x1="23.415" y1="30.845" x2="23.415" y2="26.845" width="0" layer="19" extent="1-1"/>
 <wire x1="23.415" y1="33.345" x2="23.415" y2="30.845" width="0" layer="19" extent="1-1"/>
@@
 <wire x1="-28.885" y1="-389.975" x2="-30.16" y2="-387.875" width="0" layer="19" extent="1-1"/>
 </signal>
+<signal name="NFAULT">
+<contactref element="IC1" pad="18"/>
+<contactref element="IC2" pad="18"/>
+<contactref element="U1" pad="80"/>
+<contactref element="R20" pad="1"/>
+<wire x1="-31.987" y1="-161.66" x2="-42.76" y2="-426.72" width="0" layer="19" extent="1-1"/>
+<wire x1="35.115" y1="37.545" x2="-31.987" y2="-161.66" width="0" layer="19" extent="1-1"/>
+<wire x1="69.585" y1="30.878" x2="35.115" y2="37.545" width="0" layer="19" extent="1-1"/>
+</signal>
 </signals>
