File: pcb/smd/zeta2/zeta2rework_lw_v32_rework.sch (EAGLE design)
At the start: 98 parts, among them IC1 DRV8844PWPR, IC2 DRV8844PWPR, J1 UJ2-MIBH2-4-SMT-TR, M1 IRLML2502, M2 IRLML2502, M3 IRLML2502, U1 STM32F427VI, U3 ICM-20948, U5 DS18B20U+

Commit message: progress on traces
Parts:
- added SJ3: (no value), jumper:SJ2W
- added UART2: (no value), pinhead:PINHD-1X4
Connections:
- new net M_RESET: IC1.NRESRT, IC2.NRESRT, U1.PB5
- new net N$41: P1.2, P3.2, SJ3.2
- net +3V3: now also SJ3.3; no longer IC1.NRESRT, IC2.NRESRT
- net +5V: now also SJ3.1, UART2.1
- net GND: now also UART2.4
- net M_PWM_RB: now also U1.PE5; no longer U1.PE6
- net M_PWM_RF: now also U1.PE6; no longer U1.PE5
- net N$32: no longer P1.2, P3.2
- net UART2_RX: now also UART2.3
- net UART2_TX: now also UART2.2
