File: pcb/smd/zeta2/zeta2rework_lw_v33_rework.sch (EAGLE design)
At the start: 99 parts, among them IC1 DRV8844PWPR, IC2 DRV8844PWPR, J1 UJ2-MIBH2-4-SMT-TR, M1 IRLML2502, M2 IRLML2502, M3 IRLML2502, U1 STM32F427VI, U3 ICM-20948, U5 DS18B20U+

Commit message: progress on traces
Parts:
- removed D2: BAT60JFILM, BAT60JFILM:BAT60JFILM
- removed J1: UJ2-MIBH2-4-SMT-TR, UJ2-MIBH2-4-SMT-TR:UJ2-MIBH2-4-SMT-TR
- removed R12: 1k5, rcl:R-EU_R0603
- removed R14, R18: 22r, rcl:R-EU_R0603
- removed R16: 100k, rcl:R-EU_R0603
- removed R19: 100r, rcl:R-EU_R0603
- removed SJ2: (no value), jumper:SJ
- added SJ3: (no value), jumper:SJ2W
Connections:
- removed net N$15: D2.A, J1.1
- removed net N$17: J1.4, R16.2
- removed net N$25: R19.1, SJ2.2
- removed net N$34: J1.2, R14.2
- removed net N$40: J1.SHIELD, R19.2
- removed net N$5: J1.3, R12.1, R18.2
- new net M_RESET: IC1.NRESRT, IC2.NRESRT, U1.PB5
- new net N$41: P1.2, P3.2, SJ3.2
- net +3V3: now also SJ3.3; no longer IC1.NRESRT, IC2.NRESRT, R12.2
- net +5V: now also SJ3.1; no longer D2.K
- net GND: no longer J1.5, SJ2.1
- net M_PWM_RB: now also U1.PE5; no longer U1.PE6
- net M_PWM_RF: now also U1.PE6; no longer U1.PE5
- net N$32: no longer P1.2, P3.2
- net USB_OTG_DM: no longer R14.1
- net USB_OTG_DP: no longer R18.1
- net USB_OTG_ID: no longer R16.1
